File: src/myFirstDevBoard.kicad_pcb (KiCad board)
At the start: 2 copper layers, 96.5 x 68.6 mm, 36 parts, among them J1 Conn_01x15_Male, J2 Conn_01x15_Male, Q1 BC550, Q2 BC550, Q3 BC550, SW1 SW_Push, SW2 SW_Push, SW3 SW_Push, SW4 SW_Push, SW5 SW_SLIDER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

Commit message: updating version number
Other:
- board text added: "V1.00"
- board text removed: "V0.03"
Changed lines of the file:
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@@
     )
   )
-  (gr_text V0.03 (at 10.16 71.12) (layer B.SilkS)
+  (gr_text V1.00 (at 10.16 71.12) (layer B.SilkS)
     (effects (font (size 1.5 1.5) (thickness 0.3)) (justify mirror))
   )
